Commit message: description : fix test

File: alpo_description/urdf/ros2_control/alpo.ros2_control.xacro (robot description, xacro)
@@ -10,5 +10,5 @@
         filename="$(find romea_mobile_base_description)/ros2_control/base2FWS2RWD.ros2_control.xacro" />
     </xacro:if>
-    <xacro:property name="conf" value="$(find adap2e_description)/config/adap2e_${model}.yaml" />
+    <xacro:property name="conf" value="$(find alpo_description)/config/alpo_${model}.yaml" />
     <xacro:property name="props" value="${load_yaml(conf)}" />
     <!-- Joint names -->
