Commit message: alpo description :  update alpo xacros files to support ros2_control

File: alpo_description/urdf/alpo.xacro (robot description, xacro)
@@ -3,6 +3,7 @@
   <xacro:macro name="alpo" params="model use_sim prefix">
     <xacro:include filename="$(find alpo_description)/urdf/color.xacro" />
-    <xacro:include filename="$(find romea_odo_description)/urdf/2FWS_4WD_chassis.xacro"/>
-    <xacro:property name="conf" value="$(find adap2e_description)/config/alpo_${model}.yaml" />
+    <xacro:include filename="$(find romea_mobile_base_description)/urdf/2FWS_4WD_chassis.xacro"/>
+    <xacro:include filename="$(find romea_mobile_base_description)/ros2_control/2FWS_4WD.ros2_control.xacro"/>
+    <xacro:property name="conf" value="$(find alpo_description)/config/alpo_${model}.yaml" />
     <xacro:property name="props" value="${load_yaml(conf)['/**']['ros__parameters']['base_info']}" />
     <!-- Link names -->
@@ -46,5 +47,5 @@
     <xacro:property name="body_offset_x" value="${props['control_point'][0]}" />
     <xacro:property name="body_origin_z" value="${ground_clearance + body_height/2}" />
-    <xacro:property name="body_reference_x" value="${${props['control_point'][0]}}" />
+    <xacro:property name="body_reference_x" value="${props['control_point'][0]}" />
     <!-- Steering Properties -->
     <xacro:property name="steering_angle_max_in" value="1.04"/>
@@ -52,4 +53,5 @@
     <xacro:property name="front_wheel_y_offset" value="${props['geometry']['front_axle']['wheels']['hub_carrier_offset']}" />
     <xacro:property name="rear_wheel_y_offset" value="${props['geometry']['rear_axle']['wheels']['hub_carrier_offset']}" />
+    <xacro:property name="wheel_y_offset" value="${front_wheel_y_offset}" />
     <xacro:property name="steering_link_mass" value="1" />
     <xacro:property name="steering_link_y_size" value="${wheel_y_offset}" />
@@ -71,9 +73,9 @@
     <xacro:property name="rear_wheel_mass" value="5" />
     <!-- Wheel Mounting Positions -->
-    <xacro:property name="ground_clearance" value="${chassis_props['ground_clearance']}"/>
-    <xacro:property name="front_wheel_y_offset" value="${chassis_props['hub_carrier_offset']['front']}" />
-    <xacro:property name="rear_wheel_y_offset" value="${chassis_props['hub_carrier_offset']['rear']}" />
-    <xacro:property name="front_wheel_y_offset" value="${chassis_props['hub_carrier_offset']['front']}" />
-    <xacro:property name="rear_wheel_y_offset" value="${chassis_props['hub_carrier_offset']['rear']}" />
+<!--    <xacro:property name="ground_clearance" value="${chassis_props['ground_clearance']}"/>-->
+<!--    <xacro:property name="front_wheel_y_offset" value="${chassis_props['hub_carrier_offset']['front']}" />-->
+<!--    <xacro:property name="rear_wheel_y_offset" value="${chassis_props['hub_carrier_offset']['rear']}" />-->
+<!--    <xacro:property name="front_wheel_y_offset" value="${chassis_props['hub_carrier_offset']['front']}" />-->
+<!--    <xacro:property name="rear_wheel_y_offset" value="${chassis_props['hub_carrier_offset']['rear']}" />-->
     <xacro:property name="chassis_height" value="${min(front_wheel_radius,rear_wheel_radius)}" />
     <xacro:chassis>

File: alpo_description/urdf/alpo_4x4.urdf.xacro (robot description, xacro)
@@ -5,5 +5,5 @@
   <xacro:arg name="controller_conf_yaml_file" default=""/>
   <xacro:include filename="$(find alpo_description)/urdf/alpo.xacro" />
-  <xacro:adap2e model="fat" use_sim="$(arg use_sim)" prefix="$(arg prefix)"/>
+  <xacro:alpo model="4x4" use_sim="$(arg use_sim)" prefix="$(arg prefix)"/>
   <gazebo>
     <plugin filename="libgazebo_ros2_control.so" name="gazebo_ros2_control">

File: alpo_description/urdf/alpo_slim.urdf.xacro (robot description, xacro)
@@ -4,5 +4,5 @@
   <xacro:arg name="use_sim" default="true" />
   <xacro:arg name="controller_conf_yaml_file" default=""/>
-  <xacro:include filename="$(find adap2e_description)/urdf/adap2e.xacro" />
+  <xacro:include filename="$(find alpo_description)/urdf/alpo.xacro" />
   <xacro:adap2e model="slim" use_sim="$(arg use_sim)" prefix="$(arg prefix)"/>
   <gazebo>

Commit message: alpo description : refactoring of xacro files due to changes into mobile base description package

File: alpo_description/urdf/alpo.xacro (robot description, xacro)
@@ -1,5 +1,5 @@
 <?xml version="1.0"?>
 <robot name="alpo" xmlns:xacro="http://www.ros.org/wiki/xacro">
-  <xacro:macro name="alpo" params="model use_sim prefix">
+  <xacro:macro name="alpo" params="model mode prefix">
     <xacro:include filename="$(find alpo_description)/urdf/color.xacro" />
     <xacro:include filename="$(find romea_mobile_base_description)/urdf/2FWS_4WD_chassis.xacro"/>
@@ -79,4 +79,11 @@
 <!--    <xacro:property name="rear_wheel_y_offset" value="${chassis_props['hub_carrier_offset']['rear']}" />-->
     <xacro:property name="chassis_height" value="${min(front_wheel_radius,rear_wheel_radius)}" />
+    <!-- Ros2 control hardware plugin -->
+    <xacro:if value="${model == '4x4'}">
+       <xacro:property name="simulation_hardware_plugin" value="romea_mobile_base_gazebo/GazeboSystemInterface2FWS4WD"/>
+    </xacro:if>
+    <xacro:if value="${model == 'slim'}">
+       <xacro:property name="simulation_hardware_plugin" value="romea_mobile_base_gazebo/GazeboSystemInterface2FW2RWD"/>
+    </xacro:if>
     <xacro:chassis>
       <!-- visual chassis -->
@@ -101,5 +108,7 @@
       <cylinder length="${wheel_width}" radius="${wheel_radius}"/>
     </xacro:chassis>
-     <xacro:base_control use_sim="${use_sim}"/>
+    <xacro:if value="${mode == 'simulation'}">
+       <xacro:base_control mode="${mode}"/>
+    </xacro:if>
   </xacro:macro>
 </robot>

File: alpo_description/urdf/alpo_4x4.urdf.xacro (robot description, xacro)
@@ -2,8 +2,8 @@
 <robot name="alpo_4x4" xmlns:xacro="http://www.ros.org/wiki/xacro">
   <xacro:arg name="prefix" default="" />
-  <xacro:arg name="use_sim" default="true" />
+  <xacro:arg name="mode" default="simulation" />
   <xacro:arg name="controller_conf_yaml_file" default=""/>
   <xacro:include filename="$(find alpo_description)/urdf/alpo.xacro" />
-  <xacro:alpo model="4x4" use_sim="$(arg use_sim)" prefix="$(arg prefix)"/>
+  <xacro:alpo model="4x4" mode="$(arg mode)" prefix="$(arg prefix)"/>
   <gazebo>
     <plugin filename="libgazebo_ros2_control.so" name="gazebo_ros2_control">

File: alpo_description/urdf/alpo_slim.urdf.xacro (robot description, xacro)
@@ -2,8 +2,8 @@
 <robot name="adap2e_fat" xmlns:xacro="http://www.ros.org/wiki/xacro">
   <xacro:arg name="prefix" default="" />
-  <xacro:arg name="use_sim" default="true" />
+  <xacro:arg name="mode" default="simulation" />
   <xacro:arg name="controller_conf_yaml_file" default=""/>
   <xacro:include filename="$(find alpo_description)/urdf/alpo.xacro" />
-  <xacro:adap2e model="slim" use_sim="$(arg use_sim)" prefix="$(arg prefix)"/>
+  <xacro:adap2e model="slim" mode="$(arg mode)" prefix="$(arg prefix)"/>
   <gazebo>
     <plugin filename="libgazebo_ros2_control.so" name="gazebo_ros2_control">

Commit message: alpo desctiption : change 4x4 model by fat model

File: alpo_description/urdf/alpo.xacro (robot description, xacro)
@@ -1,8 +1,14 @@
 <?xml version="1.0"?>
 <robot name="alpo" xmlns:xacro="http://www.ros.org/wiki/xacro">
-  <xacro:macro name="alpo" params="model mode prefix">
+ <xacro:macro name="alpo" params="model mode prefix">
     <xacro:include filename="$(find alpo_description)/urdf/color.xacro" />
-    <xacro:include filename="$(find romea_mobile_base_description)/urdf/2FWS_4WD_chassis.xacro"/>
-    <xacro:include filename="$(find romea_mobile_base_description)/ros2_control/2FWS_4WD.ros2_control.xacro"/>
+    <xacro:if value="${model == 'fat'}">
+       <xacro:include filename="$(find romea_mobile_base_description)/urdf/2FWS_4WD_chassis.xacro"/>
+       <xacro:include filename="$(find romea_mobile_base_description)/ros2_control/2FWS_4WD.ros2_control.xacro"/>
+    </xacro:if>
+    <xacro:if value="${model == 'slim'}">
+      <xacro:include filename="$(find romea_mobile_base_description)/urdf/2FWS_2RWD_chassis.xacro"/>
+      <xacro:include filename="$(find romea_mobile_base_description)/ros2_control/2FWS_2RWD.ros2_control.xacro"/>
+    </xacro:if>
     <xacro:property name="conf" value="$(find alpo_description)/config/alpo_${model}.yaml" />
     <xacro:property name="props" value="${load_yaml(conf)['/**']['ros__parameters']['base_info']}" />
@@ -66,7 +72,12 @@
     <xacro:property name="wheel_radius" value="${front_wheel_radius}" />
     <xacro:property name="wheel_width" value="${front_wheel_width}" />
-    <xacro:property name="minimal_wheel_steering_angle" value="-${props['wheels_steering_control']['command']['maximal_angle']}"/>
-    <xacro:property name="maximal_wheel_steering_angle" value="${props['wheels_steering_control']['command']['maximal_angle']}"/>
-    <xacro:property name="maximal_wheel_speed" value="${props['wheels_speed_control']['command']['maximal_speed']}"/>
+    <xacro:property name="minimal_wheel_steering_angle" value="-${props['front_wheels_steering_control']['command']['maximal_angle']}"/>
+    <xacro:property name="maximal_wheel_steering_angle" value="${props['front_wheels_steering_control']['command']['maximal_angle']}"/>
+    <xacro:if value="${model == 'fat'}">
+       <xacro:property name="maximal_wheel_speed" value="${props['wheels_speed_control']['command']['maximal_speed']}"/>
+    </xacro:if>
+    <xacro:if value="${model == 'slim'}">
+       <xacro:property name="maximal_wheel_speed" value="${props['rear_wheels_speed_control']['command']['maximal_speed']}"/>
+    </xacro:if>
     <xacro:property name="wheel_mass" value="5" />
     <xacro:property name="front_wheel_mass" value="5" />
@@ -80,5 +91,5 @@
     <xacro:property name="chassis_height" value="${min(front_wheel_radius,rear_wheel_radius)}" />
     <!-- Ros2 control hardware plugin -->
-    <xacro:if value="${model == '4x4'}">
+    <xacro:if value="${model == 'fat'}">
        <xacro:property name="simulation_hardware_plugin" value="romea_mobile_base_gazebo/GazeboSystemInterface2FWS4WD"/>
     </xacro:if>

File: alpo_description/urdf/alpo_fat.urdf.xacro (robot description, xacro)
@@ -1,9 +1,9 @@
 <?xml version='1.0' encoding='utf-8'?>
-<robot name="alpo_4x4" xmlns:xacro="http://www.ros.org/wiki/xacro">
+<robot name="alpo_fat" xmlns:xacro="http://www.ros.org/wiki/xacro">
   <xacro:arg name="prefix" default="" />
   <xacro:arg name="mode" default="simulation" />
   <xacro:arg name="controller_conf_yaml_file" default=""/>
   <xacro:include filename="$(find alpo_description)/urdf/alpo.xacro" />
-  <xacro:alpo model="4x4" mode="$(arg mode)" prefix="$(arg prefix)"/>
+  <xacro:alpo model="fat" mode="$(arg mode)" prefix="$(arg prefix)"/>
   <gazebo>
     <plugin filename="libgazebo_ros2_control.so" name="gazebo_ros2_control">

Commit message: description :  update xacro files

File: alpo_description/urdf/alpo.xacro (robot description, xacro)
@@ -4,10 +4,10 @@
     <xacro:include filename="$(find alpo_description)/urdf/color.xacro" />
     <xacro:if value="${model == 'fat'}">
-       <xacro:include filename="$(find romea_mobile_base_description)/urdf/2FWS_4WD_chassis.xacro"/>
-       <xacro:include filename="$(find romea_mobile_base_description)/ros2_control/2FWS_4WD.ros2_control.xacro"/>
+       <xacro:include filename="$(find romea_mobile_base_description)/urdf/base2FWS4WD.chassis.xacro"/>
+       <xacro:include filename="$(find romea_mobile_base_description)/ros2_control/base2FWS4WD.ros2_control.xacro"/>
     </xacro:if>
     <xacro:if value="${model == 'slim'}">
-      <xacro:include filename="$(find romea_mobile_base_description)/urdf/2FWS_2RWD_chassis.xacro"/>
-      <xacro:include filename="$(find romea_mobile_base_description)/ros2_control/2FWS_2RWD.ros2_control.xacro"/>
+      <xacro:include filename="$(find romea_mobile_base_description)/urdf/base2FWS4WD.chassis.xacro"/>
+      <xacro:include filename="$(find romea_mobile_base_description)/ros2_control/base2FWS2RWD.ros2_control.xacro"/>
     </xacro:if>
     <xacro:property name="conf" value="$(find alpo_description)/config/alpo_${model}.yaml" />
@@ -37,4 +37,7 @@
     <xacro:property name="aabb_width" value="${props['geometry']['aabb']['width']}" />
     <xacro:property name="aabb_height" value="${props['geometry']['aabb']['height']}" />
+    <xacro:property name="aabb_center_x" value="${props['geometry']['aabb']['center'][0]}" />
+    <xacro:property name="aabb_center_y" value="${props['geometry']['aabb']['center'][1]}" />
+    <xacro:property name="aabb_center_z" value="${props['geometry']['aabb']['center'][2]}" />
     <xacro:property name="wheelbase" value="${props['geometry']['axles_distance']}"/>
     <xacro:property name="front_track" value="${props['geometry']['front_axle']['wheels_distance']}"/>
@@ -48,9 +51,4 @@
     <xacro:property name="mass_center_z" value="${props['inertia']['center'][2]}" />
     <xacro:property name="ground_clearance" value="${props['geometry']['ground_clearance']}"/>
-    <xacro:property name="body_length" value="{props['geometry']['aabb']['length']}" />
-    <xacro:property name="body_width" value="${props['geometry']['aabb']['width']}" />
-    <xacro:property name="body_height" value="${props['geometry']['aabb']['height']}" />
-    <xacro:property name="body_offset_x" value="${props['control_point'][0]}" />
-    <xacro:property name="body_origin_z" value="${ground_clearance + body_height/2}" />
     <xacro:property name="body_reference_x" value="${props['control_point'][0]}" />
     <!-- Steering Properties -->
@@ -83,10 +81,4 @@
     <xacro:property name="front_wheel_mass" value="5" />
     <xacro:property name="rear_wheel_mass" value="5" />
-    <!-- Wheel Mounting Positions -->
-<!--    <xacro:property name="ground_clearance" value="${chassis_props['ground_clearance']}"/>-->
-<!--    <xacro:property name="front_wheel_y_offset" value="${chassis_props['hub_carrier_offset']['front']}" />-->
-<!--    <xacro:property name="rear_wheel_y_offset" value="${chassis_props['hub_carrier_offset']['rear']}" />-->
-<!--    <xacro:property name="front_wheel_y_offset" value="${chassis_props['hub_carrier_offset']['front']}" />-->
-<!--    <xacro:property name="rear_wheel_y_offset" value="${chassis_props['hub_carrier_offset']['rear']}" />-->
     <xacro:property name="chassis_height" value="${min(front_wheel_radius,rear_wheel_radius)}" />
     <!-- Ros2 control hardware plugin -->
@@ -97,11 +89,18 @@
        <xacro:property name="simulation_hardware_plugin" value="romea_mobile_base_gazebo/GazeboSystemInterface2FW2RWD"/>
     </xacro:if>
+   <!-- Mesh scale -->
+    <xacro:if value="${model == 'fat' and mesh == True}">
+       <xacro:property name="mesh_scale_y" value="1.0"/>
+    </xacro:if>
+    <xacro:if value="${model == 'slim' and mesh == True}">
+       <xacro:property name="mesh_scale_y" value="0.7"/>
+    </xacro:if>
     <xacro:chassis>
       <!-- visual chassis -->
       <visual>
         <xacro:if value="${mesh == False}">
-          <origin xyz="${body_offset_x} 0 ${body_origin_z - wheel_radius}" rpy="0 0 0" />
+          <origin xyz="${aabb_center_x-body_reference_x} ${aabb_center_y}  ${aabb_center_z-chassis_height}" rpy="0 0 0" />
           <geometry>
-            <box size="${body_length} ${body_width} ${body_height}"/>
+            <box size="${aabb_length} ${aabb_width} ${aabb_height}"/>
           </geometry>
         </xacro:if>
@@ -109,5 +108,5 @@
           <origin xyz="0 0 0" rpy="0 0 ${-pi/2}" />
           <geometry>
-            <mesh filename="package://alpo_description/meshes/chassis.dae"/>
+            <mesh filename="package://alpo_description/meshes/chassis.dae" scale="1.0 ${mesh_scale_y} 1.0" />
           </geometry>
         </xacro:if>

File: alpo_description/urdf/alpo_slim.urdf.xacro (robot description, xacro)
@@ -1,9 +1,9 @@
 <?xml version='1.0' encoding='utf-8'?>
-<robot name="adap2e_fat" xmlns:xacro="http://www.ros.org/wiki/xacro">
+<robot name="alpo_slim" xmlns:xacro="http://www.ros.org/wiki/xacro">
   <xacro:arg name="prefix" default="" />
   <xacro:arg name="mode" default="simulation" />
   <xacro:arg name="controller_conf_yaml_file" default=""/>
   <xacro:include filename="$(find alpo_description)/urdf/alpo.xacro" />
-  <xacro:adap2e model="slim" mode="$(arg mode)" prefix="$(arg prefix)"/>
+  <xacro:alpo model="slim" mode="$(arg mode)" prefix="$(arg prefix)"/>
   <gazebo>
     <plugin filename="libgazebo_ros2_control.so" name="gazebo_ros2_control">

Commit message: alpo descriptions : update xacro files

File: alpo_description/urdf/alpo.xacro (robot description, xacro)
@@ -64,4 +64,6 @@
     <xacro:property name="steering_link_xz" value="0.1" />
     <!-- Wheel Properties -->
+    <xacro:property name="front_hub_carrier_offset" value="${props['geometry']['front_axle']['wheels']['hub_carrier_offset']}" />
+    <xacro:property name="rear_hub_carrier_offset" value="${props['geometry']['rear_axle']['wheels']['hub_carrier_offset']}" />
     <xacro:property name="front_wheel_radius" value="${props['geometry']['front_axle']['wheels']['radius']}" />
     <xacro:property name="rear_wheel_radius" value="${props['geometry']['rear_axle']['wheels']['radius']}" />
@@ -85,7 +87,9 @@
     <xacro:if value="${model == 'fat'}">
        <xacro:property name="simulation_hardware_plugin" value="romea_mobile_base_gazebo/GazeboSystemInterface2FWS4WD"/>
+       <xacro:property name="live_hardware_plugin" value="alpo_hardware/AlpoHardware2FWS4WD"/>
     </xacro:if>
     <xacro:if value="${model == 'slim'}">
        <xacro:property name="simulation_hardware_plugin" value="romea_mobile_base_gazebo/GazeboSystemInterface2FW2RWD"/>
+       <xacro:property name="live_hardware_plugin" value="alpo_hardware/AlpoHardware2FWS2RWD"/>
     </xacro:if>
    <!-- Mesh scale -->
@@ -118,5 +122,5 @@
       <cylinder length="${wheel_width}" radius="${wheel_radius}"/>
     </xacro:chassis>
-    <xacro:if value="${mode == 'simulation'}">
+    <xacro:if value="${mode == 'simulation' or mode == 'live'}">
        <xacro:base_control mode="${mode}"/>
     </xacro:if>

Commit message: alpo description : fix mesh scale for slim alpo

File: alpo_description/urdf/alpo.xacro (robot description, xacro)
@@ -90,13 +90,13 @@
     </xacro:if>
     <xacro:if value="${model == 'slim'}">
-       <xacro:property name="simulation_hardware_plugin" value="romea_mobile_base_gazebo/GazeboSystemInterface2FW2RWD"/>
+       <xacro:property name="simulation_hardware_plugin" value="romea_mobile_base_gazebo/GazeboSystemInterface2FWS2RWD"/>
        <xacro:property name="live_hardware_plugin" value="alpo_hardware/AlpoHardware2FWS2RWD"/>
     </xacro:if>
    <!-- Mesh scale -->
     <xacro:if value="${model == 'fat' and mesh == True}">
-       <xacro:property name="mesh_scale_y" value="1.0"/>
+       <xacro:property name="mesh_scale_x" value="1.0"/>
     </xacro:if>
     <xacro:if value="${model == 'slim' and mesh == True}">
-       <xacro:property name="mesh_scale_y" value="0.7"/>
+       <xacro:property name="mesh_scale_x" value="0.7"/>
     </xacro:if>
     <xacro:chassis>
@@ -112,5 +112,5 @@
           <origin xyz="0 0 0" rpy="0 0 ${-pi/2}" />
           <geometry>
-            <mesh filename="package://alpo_description/meshes/chassis.dae" scale="1.0 ${mesh_scale_y} 1.0" />
+            <mesh filename="package://alpo_description/meshes/chassis.dae" scale="${mesh_scale_x} 1.0 1.0" />
           </geometry>
         </xacro:if>

Commit message: description: refactoring of robot description + add teleop configuration

File: alpo_description/urdf/alpo.xacro (robot description, xacro)
@@ -12,5 +12,5 @@
     </xacro:if>
     <xacro:property name="conf" value="$(find alpo_description)/config/alpo_${model}.yaml" />
-    <xacro:property name="props" value="${load_yaml(conf)['/**']['ros__parameters']['base_info']}" />
+    <xacro:property name="props" value="${load_yaml(conf)}" />
     <!-- Link names -->
     <xacro:property name="base_link" value="${props['links']['base_link_name']}" />
