Commit message: description replace meshes

File: alpo_description/urdf/alpo.xacro (robot description, xacro)
@@ -3,15 +3,12 @@
    <xacro:macro name="alpo" params="model mode prefix">
       <xacro:include filename="$(find alpo_description)/urdf/color.xacro" />
+      <xacro:include filename="$(find alpo_description)/urdf/half_leg.xacro" />
       <xacro:if value="${model == 'fat'}">
          <xacro:include
             filename="$(find romea_mobile_base_description)/urdf/base2FWSxxx.chassis.xacro" />
-         <!-- <xacro:include
-            filename="$(find romea_mobile_base_description)/ros2_control/base2FWS4WD.ros2_control.xacro" /> -->
       </xacro:if>
       <xacro:if value="${model == 'slim'}">
          <xacro:include
             filename="$(find romea_mobile_base_description)/urdf/base2FWSxxx.chassis.xacro" />
-         <!-- <xacro:include
-            filename="$(find romea_mobile_base_description)/ros2_control/base2FWS2RWD.ros2_control.xacro" /> -->
       </xacro:if>
       <xacro:property name="conf" value="$(find alpo_description)/config/alpo_${model}.yaml" />
@@ -58,9 +55,12 @@
       <xacro:property name="aabb_center_y" value="${props['geometry']['aabb']['center'][1]}" />
       <xacro:property name="aabb_center_z" value="${props['geometry']['aabb']['center'][2]}" />
-      <xacro:property name="wheelbase" value="${props['geometry']['axles_distance']}" />
+      <xacro:property name="wheelbase"
+         value="${props['geometry']['axles_distance']}" />
       <xacro:property name="front_track"
          value="${props['geometry']['front_axle']['wheels_distance']}" />
-      <xacro:property name="rear_track" value="${props['geometry']['rear_axle']['wheels_distance']}" />
-      <xacro:property name="track" value="${front_track}" />
+      <xacro:property name="rear_track"
+         value="${props['geometry']['rear_axle']['wheels_distance']}" />
+      <xacro:property name="track"
+         value="${front_track}" />
       <xacro:property name="ground_clearance" value="${chassis_props['ground_clearance']}" />
       <xacro:property name="mass_body" value="${props['inertia']['mass']}" />
@@ -115,22 +115,11 @@
       <xacro:property name="rear_wheel_mass" value="5" />
       <xacro:property name="chassis_height" value="${min(front_wheel_radius,rear_wheel_radius)}" />
-      <!-- Ros2 control hardware plugin -->
-      <!-- <xacro:if value="${model == 'fat'}">
-         <xacro:property name="simulation_hardware_plugin"
-            value="romea_mobile_base_gazebo/GazeboSystemInterface2FWS4WD" />
-         <xacro:property name="live_hardware_plugin" value="alpo_hardware/AlpoHardware2FWS4WD" />
-      </xacro:if>
-      <xacro:if value="${model == 'slim'}">
-         <xacro:property name="simulation_hardware_plugin"
-            value="romea_mobile_base_gazebo/GazeboSystemInterface2FWS2RWD" />
-         <xacro:property name="live_hardware_plugin" value="alpo_hardware/AlpoHardware2FWS2RWD" />
-      </xacro:if> -->
       <!-- Mesh scale -->
-      <xacro:if value="${model == 'fat' and mesh == True}">
+      <!-- <xacro:if value="${model == 'fat' and mesh == True}">
          <xacro:property name="mesh_scale_x" value="1.0" />
       </xacro:if>
       <xacro:if value="${model == 'slim' and mesh == True}">
          <xacro:property name="mesh_scale_x" value="0.7" />
-      </xacro:if>
+      </xacro:if> -->
       <xacro:chassis>
          <!-- visual chassis -->
@@ -147,6 +136,12 @@
                <origin xyz="0 0 0" rpy="0 0 ${-pi/2}" />
                <geometry>
-                  <mesh filename="package://alpo_description/meshes/chassis.dae"
-                     scale="${mesh_scale_x} 1.0 1.0" />
+                  <xacro:if value="${model == 'fat'}">
+                     <mesh filename="package://alpo_description/meshes/pom_4x4.obj" />
+                  </xacro:if>
+                  <xacro:if value="${model == 'slim'}">
+                     <mesh filename="package://alpo_description/meshes/pom_slim.obj" />
+                  </xacro:if>
+                  <!-- <mesh filename="package://alpo_description/meshes/chassis.dae"
+                     scale="${mesh_scale_x} 1.0 1.0" /> -->
                </geometry>
             </xacro:if>
@@ -158,4 +153,13 @@
          <cylinder length="${wheel_width}" radius="${wheel_radius}" />
       </xacro:chassis>
+      <xacro:if value="${mesh == True}">
+         <xacro:half_leg side="left">
+            <origin xyz="1.5 ${aabb_width / 2 - 0.32} -0.032" rpy="-1.6525 0 ${pi/2}" />
+         </xacro:half_leg>
+         <xacro:half_leg side="right">
+            <origin xyz="1.5 ${-aabb_width / 2} -0.032" rpy="-1.6525 0 ${pi/2}" />
+         </xacro:half_leg>
+      </xacro:if>
+      <xacro:pom_gazebo_material link="${prefix}${base_link}" />
       <!-- <xacro:if value="${mode == 'simulation' or mode == 'live'}">
          <xacro:base_control mode="${mode}" />

File: alpo_description/urdf/color.xacro (robot description, xacro)
@@ -3,5 +3,5 @@
     <xacro:macro name="beige" params="">
         <material name="beige">
-            <color rgba="0.89 0.86 0.78 1"/>
+            <color rgba="0.89 0.86 0.78 1" />
         </material>
     </xacro:macro>
@@ -9,10 +9,11 @@
         <gazebo reference="${link}">
             <visual>
-                <material>
-                    <ambient>0.89 0.86 0.78 1</ambient>
-                    <diffuse>0.89 0.86 0.78 1</diffuse>
-                    <specular>0 0 0 0</specular>
-                    <emissive>0 0 0 1</emissive>
-                </material>
+                <lighting>1</lighting>
+                <!-- <material> -->
+                <!-- <ambient>0.89 0.86 0.78 1</ambient> -->
+                <!-- <diffuse>0.89 0.86 0.78 1</diffuse> -->
+                <!-- <specular>0 0 0 0</specular> -->
+                <!-- <emissive>0 0 0 1</emissive> -->
+                <!-- </material> -->
             </visual>
         </gazebo>
@@ -20,5 +21,5 @@
     <xacro:macro name="brown" params="">
         <material name="brown">
-            <color rgba="0.4 0.27 0.18 1"/>
+            <color rgba="0.4 0.27 0.18 1" />
         </material>
     </xacro:macro>
@@ -35,3 +36,15 @@
         </gazebo>
     </xacro:macro>
+    <xacro:macro name="pom_gazebo_material" params="link">
+        <gazebo reference="${link}">
+            <visual>
+                <material>
+                    <script>
+                        <uri>package://alpo_description/meshes/pom.material</uri>
+                        <name>alpo/pom</name>
+                    </script>
+                </material>
+            </visual>
+        </gazebo>
+    </xacro:macro>
 </robot>

File: alpo_description/urdf/half_leg.xacro (robot description, xacro)
@@ -8,11 +8,11 @@
                 <origin xyz="0 0 0" rpy="0 0 0" />
                 <geometry>
-                    <mesh filename="package://alpo_description/meshes/half_leg.dae"/>
+                    <mesh filename="package://alpo_description/meshes/half_leg.obj" />
                 </geometry>
-                <xacro:beige/>
+                <xacro:beige />
             </visual>
         </link>
         <joint name="${prefix}half_leg_${side}_joint" type="fixed">
-            <xacro:insert_block name="joint_origin"/>
+            <xacro:insert_block name="joint_origin" />
             <parent link="${prefix}base_link" />
             <child link="${prefix}half_leg_${side}_link" />

Commit message: description: update xacro file in order to load front and rear wheels visuals
Signed-off-by: Jean Laneurit <jean.laneurit@inrae.fr>

File: alpo_description/urdf/alpo.xacro (robot description, xacro)
@@ -97,6 +97,4 @@
       <xacro:property name="rear_wheel_width"
          value="${props['geometry']['rear_axle']['wheels']['width']}" />
-      <xacro:property name="wheel_radius" value="${front_wheel_radius}" />
-      <xacro:property name="wheel_width" value="${front_wheel_width}" />
       <xacro:property name="minimal_wheel_steering_angle"
          value="-${props['front_wheels_steering_control']['command']['maximal_angle']}" />
@@ -111,5 +109,5 @@
             value="${props['rear_wheels_speed_control']['command']['maximal_speed']}" />
       </xacro:if>
-      <xacro:property name="wheel_mass" value="5" />
+      <!-- <xacro:property name="wheel_mass" value="5" /> -->
       <xacro:property name="front_wheel_mass" value="5" />
       <xacro:property name="rear_wheel_mass" value="5" />
@@ -142,6 +140,4 @@
                      <mesh filename="package://alpo_description/meshes/pom_slim.obj" />
                   </xacro:if>
-                  <!-- <mesh filename="package://alpo_description/meshes/chassis.dae"
-                     scale="${mesh_scale_x} 1.0 1.0" /> -->
                </geometry>
             </xacro:if>
@@ -150,6 +146,8 @@
          <!-- visual front steering -->
          <box size="${steering_link_xz_size} ${steering_link_y_size} ${steering_link_xz_size}" />
-         <!-- visual wheel -->
-         <cylinder length="${wheel_width}" radius="${wheel_radius}" />
+         <!-- visual front wheel -->
+         <cylinder length="${front_wheel_width}" radius="${front_wheel_radius}" />
+         <!-- visual rear wheel -->
+         <cylinder length="${rear_wheel_width}" radius="${rear_wheel_radius}" />
       </xacro:chassis>
       <xacro:if value="${mesh == True}">
@@ -162,7 +160,4 @@
       </xacro:if>
       <xacro:pom_gazebo_material link="${prefix}${base_link}" />
-      <!-- <xacro:if value="${mode == 'simulation' or mode == 'live'}">
-         <xacro:base_control mode="${mode}" />
-      </xacro:if> -->
    </xacro:macro>
 </robot>

Commit message: description: update xacro
Signed-off-by: Jean Laneurit <jean.laneurit@inrae.fr>

File: alpo_description/urdf/alpo.xacro (robot description, xacro)
@@ -49,10 +49,16 @@
       <xacro:property name="mesh" value="True" />
       <!-- Base Properties -->
-      <xacro:property name="aabb_length" value="${props['geometry']['aabb']['length']}" />
-      <xacro:property name="aabb_width" value="${props['geometry']['aabb']['width']}" />
-      <xacro:property name="aabb_height" value="${props['geometry']['aabb']['height']}" />
-      <xacro:property name="aabb_center_x" value="${props['geometry']['aabb']['center'][0]}" />
-      <xacro:property name="aabb_center_y" value="${props['geometry']['aabb']['center'][1]}" />
-      <xacro:property name="aabb_center_z" value="${props['geometry']['aabb']['center'][2]}" />
+      <xacro:property name="aabb_length"
+         value="${props['geometry']['aabb']['length']}" />
+      <xacro:property name="aabb_width"
+         value="${props['geometry']['aabb']['width']}" />
+      <xacro:property name="aabb_height"
+         value="${props['geometry']['aabb']['height']}" />
+      <xacro:property name="aabb_center_x"
+         value="${props['geometry']['aabb']['center'][0]}" />
+      <xacro:property name="aabb_center_y"
+         value="${props['geometry']['aabb']['center'][1]}" />
+      <xacro:property name="aabb_center_z"
+         value="${props['geometry']['aabb']['center'][2]}" />
       <xacro:property name="wheelbase"
          value="${props['geometry']['axles_distance']}" />
@@ -63,25 +69,18 @@
       <xacro:property name="track"
          value="${front_track}" />
-      <xacro:property name="ground_clearance" value="${chassis_props['ground_clearance']}" />
-      <xacro:property name="mass_body" value="${props['inertia']['mass']}" />
-      <xacro:property name="mass_base" value="${props['inertia']['mass']}" />
-      <xacro:property name="mass_center_x" value="${props['inertia']['center'][0]}" />
-      <xacro:property name="mass_center_y" value="${props['inertia']['center'][1]}" />
-      <xacro:property name="mass_center_z" value="${props['inertia']['center'][2]}" />
-      <xacro:property name="ground_clearance" value="${props['geometry']['ground_clearance']}" />
-      <xacro:property name="body_reference_x" value="${props['control_point'][0]}" />
-      <!-- Steering Properties -->
-      <xacro:property name="steering_angle_max_in" value="1.04" />
-      <xacro:property name="steering_angle_max_out" value="0.59" />
-      <xacro:property name="front_wheel_y_offset"
-         value="${props['geometry']['front_axle']['wheels']['hub_carrier_offset']}" />
-      <xacro:property name="rear_wheel_y_offset"
-         value="${props['geometry']['rear_axle']['wheels']['hub_carrier_offset']}" />
-      <xacro:property name="wheel_y_offset" value="${front_wheel_y_offset}" />
-      <xacro:property name="steering_link_mass" value="1" />
-      <xacro:property name="steering_link_y_size" value="${wheel_y_offset}" />
-      <xacro:property name="steering_link_xz_size" value="0.1" />
-      <xacro:property name="steering_link_y" value="${wheel_y_offset}" />
-      <xacro:property name="steering_link_xz" value="0.1" />
+      <xacro:property name="mass_body"
+         value="${props['inertia']['mass']}" />
+      <xacro:property name="mass_base"
+         value="${props['inertia']['mass']}" />
+      <xacro:property name="mass_center_x"
+         value="${props['inertia']['center'][0]}" />
+      <xacro:property name="mass_center_y"
+         value="${props['inertia']['center'][1]}" />
+      <xacro:property name="mass_center_z"
+         value="${props['inertia']['center'][2]}" />
+      <xacro:property name="ground_clearance"
+         value="${props['geometry']['ground_clearance']}" />
+      <xacro:property name="body_reference_x"
+         value="${props['control_point'][0]}" />
       <!-- Wheel Properties -->
       <xacro:property name="front_hub_carrier_offset"
@@ -97,8 +96,6 @@
       <xacro:property name="rear_wheel_width"
          value="${props['geometry']['rear_axle']['wheels']['width']}" />
-      <xacro:property name="minimal_wheel_steering_angle"
-         value="-${props['front_wheels_steering_control']['command']['maximal_angle']}" />
-      <xacro:property name="maximal_wheel_steering_angle"
-         value="${props['front_wheels_steering_control']['command']['maximal_angle']}" />
+      <xacro:property name="chassis_height"
+         value="${min(front_wheel_radius,rear_wheel_radius)}" />
       <xacro:if value="${model == 'fat'}">
          <xacro:property name="maximal_wheel_speed"
@@ -109,15 +106,14 @@
             value="${props['rear_wheels_speed_control']['command']['maximal_speed']}" />
       </xacro:if>
-      <!-- <xacro:property name="wheel_mass" value="5" /> -->
       <xacro:property name="front_wheel_mass" value="5" />
       <xacro:property name="rear_wheel_mass" value="5" />
-      <xacro:property name="chassis_height" value="${min(front_wheel_radius,rear_wheel_radius)}" />
-      <!-- Mesh scale -->
-      <!-- <xacro:if value="${model == 'fat' and mesh == True}">
-         <xacro:property name="mesh_scale_x" value="1.0" />
-      </xacro:if>
-      <xacro:if value="${model == 'slim' and mesh == True}">
-         <xacro:property name="mesh_scale_x" value="0.7" />
-      </xacro:if> -->
+      <!-- Steering Properties -->
+      <xacro:property name="minimal_wheel_steering_angle"
+         value="-${props['front_wheels_steering_control']['command']['maximal_angle']}" />
+      <xacro:property name="maximal_wheel_steering_angle"
+         value="${props['front_wheels_steering_control']['command']['maximal_angle']}" />
+      <xacro:property name="front_wheel_steering_link_mass" value="1" />
+      <xacro:property name="front_wheel_steering_link_y" value="${front_hub_carrier_offset}" />
+      <xacro:property name="front_wheel_steering_link_xz" value="0.05" />
       <xacro:chassis>
          <!-- visual chassis -->
@@ -145,5 +141,5 @@
          </visual>
          <!-- visual front steering -->
-         <box size="${steering_link_xz_size} ${steering_link_y_size} ${steering_link_xz_size}" />
+         <box size="${front_wheel_steering_link_xz} ${front_wheel_steering_link_y} ${front_wheel_steering_link_xz}" />
          <!-- visual front wheel -->
          <cylinder length="${front_wheel_width}" radius="${front_wheel_radius}" />

Commit message: refactoring yaml and xacro files
Signed-off-by: jean.laneurit <jean.laneurit@inrae.fr>

File: alpo_description/urdf/alpo.xacro (robot description, xacro)
@@ -141,5 +141,6 @@
          </visual>
          <!-- visual front steering -->
-         <box size="${front_wheel_steering_link_xz} ${front_wheel_steering_link_y} ${front_wheel_steering_link_xz}" />
+         <box
+            size="${front_wheel_steering_link_xz} ${front_wheel_steering_link_y} ${front_wheel_steering_link_xz}" />
          <!-- visual front wheel -->
          <cylinder length="${front_wheel_width}" radius="${front_wheel_radius}" />

Commit message: description: change way to define visuals into xacro files
Signed-off-by: jean.laneurit <jean.laneurit@inrae.fr>

File: alpo_description/urdf/alpo.xacro (robot description, xacro)
@@ -2,6 +2,4 @@
 <robot name="alpo" xmlns:xacro="http://www.ros.org/wiki/xacro">
    <xacro:macro name="alpo" params="model mode prefix">
-      <xacro:include filename="$(find alpo_description)/urdf/color.xacro" />
-      <xacro:include filename="$(find alpo_description)/urdf/half_leg.xacro" />
       <xacro:if value="${model == 'fat'}">
          <xacro:include
@@ -12,11 +10,18 @@
             filename="$(find romea_mobile_base_description)/urdf/base2FWSxxx.chassis.xacro" />
       </xacro:if>
+      <xacro:include filename="$(find alpo_description)/urdf/visual/color.xacro" />
+      <xacro:include filename="$(find alpo_description)/urdf/visual/half_leg.xacro" />
+      <xacro:include filename="$(find alpo_description)/urdf/visual/chassis.xacro" />
+      <xacro:include filename="$(find alpo_description)/urdf/visual/wheels.xacro" />
+      <xacro:include filename="$(find alpo_description)/urdf/visual/arms.xacro" />
       <xacro:property name="conf" value="$(find alpo_description)/config/alpo_${model}.yaml" />
       <xacro:property name="props" value="${load_yaml(conf)}" />
       <!-- Link names -->
-      <xacro:property name="base_link" value="${props['links']['base_link_name']}" />
+      <xacro:property name="base_link"
+         value="${props['links']['base_link_name']}" />
       <xacro:property name="base_footprint_link"
          value="${props['links']['base_footprint_link_name']}" />
-      <xacro:property name="inertial_link" value="${props['links']['inertial_link_name']}" />
+      <xacro:property name="inertial_link"
+         value="${props['links']['inertial_link_name']}" />
       <xacro:property name="front_left_wheel_steering_link"
          value="${props['links']['front_left_wheel_steering_link_name']}" />
@@ -84,4 +89,5 @@
          value="${props['control_point'][0]}" />
       <!-- Wheel Properties -->
+      <xacro:property name="front_wheel_x_offset" value="0.0" />
       <xacro:property name="front_hub_carrier_offset"
          value="${props['geometry']['front_axle']['wheels']['hub_carrier_offset']}" />
@@ -117,34 +123,11 @@
       <xacro:property name="front_wheel_steering_link_xz" value="0.05" />
       <xacro:chassis>
-         <!-- visual chassis -->
-         <visual>
-            <xacro:if value="${mesh == False}">
-               <origin
-                  xyz="${aabb_center_x-body_reference_x} ${aabb_center_y}  ${aabb_center_z-chassis_height}"
-                  rpy="0 0 0" />
-               <geometry>
-                  <box size="${aabb_length} ${aabb_width} ${aabb_height}" />
-               </geometry>
-            </xacro:if>
-            <xacro:if value="${mesh == True}">
-               <origin xyz="0 0 0" rpy="0 0 ${-pi/2}" />
-               <geometry>
-                  <xacro:if value="${model == 'fat'}">
-                     <mesh filename="package://alpo_description/meshes/pom_4x4.obj" />
-                  </xacro:if>
-                  <xacro:if value="${model == 'slim'}">
-                     <mesh filename="package://alpo_description/meshes/pom_slim.obj" />
-                  </xacro:if>
-               </geometry>
-            </xacro:if>
-            <xacro:beige />
-         </visual>
-         <!-- visual front steering -->
-         <box
-            size="${front_wheel_steering_link_xz} ${front_wheel_steering_link_y} ${front_wheel_steering_link_xz}" />
-         <!-- visual front wheel -->
-         <cylinder length="${front_wheel_width}" radius="${front_wheel_radius}" />
-         <!-- visual rear wheel -->
-         <cylinder length="${rear_wheel_width}" radius="${rear_wheel_radius}" />
+         <xacro:chassis_visual />
+         <xacro:front_left_arm_visual />
+         <xacro:front_right_arm_visual />
+         <xacro:front_left_wheel_visual />
+         <xacro:front_right_wheel_visual />
+         <xacro:rear_left_wheel_visual />
+         <xacro:rear_right_wheel_visual />
       </xacro:chassis>
       <xacro:if value="${mesh == True}">

Commit message: Fix wheel mass to avoid crazy robot in simulation
- Set mass more realistic
- The mass of the steering link should be greater than the wheel link

File: alpo_description/urdf/alpo.xacro (robot description, xacro)
@@ -112,6 +112,6 @@
             value="${props['rear_wheels_speed_control']['command']['maximal_speed']}" />
       </xacro:if>
-      <xacro:property name="front_wheel_mass" value="5" />
-      <xacro:property name="rear_wheel_mass" value="5" />
+      <xacro:property name="front_wheel_mass" value="10" />
+      <xacro:property name="rear_wheel_mass" value="10" />
       <!-- Steering Properties -->
       <xacro:property name="minimal_wheel_steering_angle"
@@ -119,5 +119,5 @@
       <xacro:property name="maximal_wheel_steering_angle"
          value="${props['front_wheels_steering_control']['command']['maximal_angle']}" />
-      <xacro:property name="front_wheel_steering_link_mass" value="1" />
+      <xacro:property name="front_wheel_steering_link_mass" value="25" />
       <xacro:property name="front_wheel_steering_link_y" value="${front_hub_carrier_offset}" />
       <xacro:property name="front_wheel_steering_link_xz" value="0.05" />
