Commit message: description:  add missing properties into ros2_control xacro file
Signed-off-by: jean.laneurit <jean.laneurit@inrae.fr>

File: alpo_description/ros2_control/alpo.ros2_control.xacro (robot description, xacro)
@@ -43,4 +43,14 @@
     <xacro:property name="rear_hub_carrier_offset"
       value="${props['geometry']['rear_axle']['wheels']['hub_carrier_offset']}" />
+    <xacro:property name="maximal_wheel_steering_angle"
+      value="${props['front_wheels_steering_control']['command']['maximal_angle']}" />
+    <xacro:if value="${model == 'fat'}">
+      <xacro:property name="maximal_wheel_speed"
+        value="${props['wheels_speed_control']['command']['maximal_speed']}" />
+    </xacro:if>
+    <xacro:if value="${model == 'slim'}">
+      <xacro:property name="maximal_wheel_speed"
+        value="${props['rear_wheels_speed_control']['command']['maximal_speed']}" />
+    </xacro:if>
     <!-- simulation plugins -->
     <xacro:if value="${model == 'fat'}">

Commit message: add support of isaac sim
Signed-off-by: jean.laneurit <jean.laneurit@inrae.fr>

File: alpo_description/ros2_control/alpo.ros2_control.xacro (robot description, xacro)
@@ -54,13 +54,37 @@
     </xacro:if>
     <!-- simulation plugins -->
-    <xacro:if value="${model == 'fat'}">
-      <xacro:property name="simulation_hardware_plugin"
-        value="romea_mobile_base_gazebo/GazeboSystemInterface2FWS4WD" />
-      <xacro:property name="live_hardware_plugin" value="alpo_hardware/AlpoHardware2FWS4WD" />
+    <xacro:if value="${'simulation' in mode}">
+      <xacro:if value="${'gazebo' in  mode}">
+        <xacro:if value="${model == 'fat'}">
+          <xacro:property
+            name="simulation_hardware_plugin"
+            value="romea_mobile_base_gazebo/GazeboSystemInterface2FWS4WD" />
+        </xacro:if>
+        <xacro:if value="${model == 'slim'}">
+          <xacro:property
+            name="simulation_hardware_plugin"
+            value="romea_mobile_base_gazebo/GazeboSystemInterface2FWS2RWD" />
+        </xacro:if>
+      </xacro:if>
+      <xacro:if value="${'4dv' in  mode or 'isaac' in mode}">
+        <xacro:if value="${model == 'fat'}">
+          <xacro:property
+            name="simulation_hardware_plugin"
+            value="romea_mobile_base_simulation/GenericSimulationSystemInterface2FWS4WD" />
+        </xacro:if>
+        <xacro:if value="${model == 'slim'}">
+          <xacro:property
+            name="simulation_hardware_plugin"
+            value="romea_mobile_base_simulation/GenericSimulationSystemInterface2FWS2RWD" />
+        </xacro:if>
+      </xacro:if>
     </xacro:if>
-    <xacro:if value="${model == 'slim'}">
-      <xacro:property name="simulation_hardware_plugin"
-        value="romea_mobile_base_gazebo/GazeboSystemInterface2FWS2RWD" />
-      <xacro:property name="live_hardware_plugin" value="alpo_hardware/AlpoHardware2FWS2RWD" />
+    <xacro:if value="${mode ==  'live'}">
+      <xacro:if value="${model == 'fat'}">
+        <xacro:property name="live_hardware_plugin" value="alpo_hardware/AlpoHardware2FWS4WD" />
+      </xacro:if>
+      <xacro:if value="${model == 'slim'}">
+        <xacro:property name="live_hardware_plugin" value="alpo_hardware/AlpoHardware2FWS2RWD" />
+      </xacro:if>
     </xacro:if>
     <xacro:base_control mode="${mode}" base_name="${base_name}" />

File: alpo_description/urdf/alpo_fat.urdf.xacro (robot description, xacro)
@@ -9,12 +9,10 @@
   <xacro:include filename="$(find alpo_description)/urdf/alpo.xacro" />
   <xacro:alpo model="fat" mode="$(arg mode)" prefix="$(arg prefix)" />
-  <gazebo>
-    <plugin filename="libromea_gazebo_ros2_control.so" name="gazebo_ros2_control">
-      <ros2_control_config_file>$(arg ros2_control_config_urdf_file)</ros2_control_config_file>
-      <controller_manager_config_file>$(arg controller_manager_config_yaml_file)</controller_manager_config_file>
-      <ros>
-        <namespace>$(arg ros_prefix)$(arg base_name)</namespace>
-      </ros>
-    </plugin>
-  </gazebo>
+  <xacro:include filename="$(find alpo_description)/urdf/alpo.simulation.xacro" />
+  <xacro:alpo_simulation
+    mode="$(arg mode)"
+    base_name="$(arg base_name)"
+    ros_prefix="$(arg ros_prefix)"
+    ros2_control_config_urdf_file="$(arg ros2_control_config_urdf_file)"
+    controller_manager_config_yaml_file="$(arg controller_manager_config_yaml_file)" />
 </robot>

File: alpo_description/urdf/alpo_slim.urdf.xacro (robot description, xacro)
@@ -9,12 +9,10 @@
   <xacro:include filename="$(find alpo_description)/urdf/alpo.xacro" />
   <xacro:alpo model="slim" mode="$(arg mode)" prefix="$(arg prefix)" />
-  <gazebo>
-    <plugin filename="libromea_gazebo_ros2_control.so" name="gazebo_ros2_control">
-      <ros2_control_config_file>$(arg ros2_control_config_urdf_file)</ros2_control_config_file>
-      <controller_manager_config_file>$(arg controller_manager_config_yaml_file)</controller_manager_config_file>
-      <ros>
-        <namespace>$(arg ros_prefix)$(arg base_name)</namespace>
-      </ros>
-    </plugin>
-  </gazebo>
+  <xacro:include filename="$(find alpo_description)/urdf/alpo.simulation.xacro" />
+  <xacro:alpo_simulation
+    mode="$(arg mode)"
+    base_name="$(arg base_name)"
+    ros_prefix="$(arg ros_prefix)"
+    ros2_control_config_urdf_file="$(arg ros2_control_config_urdf_file)"
+    controller_manager_config_yaml_file="$(arg controller_manager_config_yaml_file)" />
 </robot>

Commit message: move deadzone handler params into yaml file

File: alpo_description/ros2_control/alpo.ros2_control.xacro (robot description, xacro)
@@ -1,4 +1,12 @@
 <?xml version="1.0"?>
 <robot name="alpo" xmlns:xacro="http://www.ros.org/wiki/xacro">
+  <!-- recursive macro to generate the list of params for hardware_options -->
+  <xacro:macro name="generate_hardware_options" params="options:=^ prefix:=^|''">
+    <xacro:if value="${options}">
+    <xacro:property name="option" value="${options.pop()}"/>
+      <param name="${prefix + option[0]}">${option[1]}</param>
+      <xacro:generate_hardware_options/>
+    </xacro:if>
+  </xacro:macro>
   <xacro:macro name="alpo_ros2_control" params="model mode prefix base_name">
     <xacro:if value="${model == 'fat'}">
@@ -11,5 +19,5 @@
     </xacro:if>
     <xacro:property name="conf" value="$(find alpo_description)/config/alpo_${model}.yaml" />
-    <xacro:property name="props" value="${load_yaml(conf)}" />
+    <xacro:property name="props" value="${xacro.load_yaml(conf)}" />
     <!-- Joint names -->
     <xacro:property name="base_footprint_joint"
@@ -45,4 +53,5 @@
     <xacro:property name="maximal_wheel_steering_angle"
       value="${props['front_wheels_steering_control']['command']['maximal_angle']}" />
+    <xacro:property name="has_deadzone_handler" value="${'deadzone_handler' in props}"/>
     <xacro:if value="${model == 'fat'}">
       <xacro:property name="maximal_wheel_speed"
@@ -88,5 +97,13 @@
       </xacro:if>
     </xacro:if>
-    <xacro:base_control mode="${mode}" base_name="${base_name}" />
+    <xacro:property name="hardware_options">
+      <param name="deadzone_enabled" value="${has_deadzone_handler}"/>
+      <xacro:if value="${has_deadzone_handler}">
+        <xacro:generate_hardware_options
+          options="${list(props['deadzone_handler'].items())}"
+          prefix="deadzone_"/>
+      </xacro:if>
+    </xacro:property>
+    <xacro:base_control mode="${mode}" base_name="${base_name}" has_hardware_options="1" />
   </xacro:macro>
 </robot>
