Commit message: refactoring
Signed-off-by: Jean Laneurit <jean.laneurit@inrae.fr>

File: pom_description/urdf/pom.simulation.xacro (robot description, xacro)
@@ -4,5 +4,5 @@
     params="mode ros_prefix base_name controller_manager_config_yaml_file">
     <xacro:if value="${'simulation' in mode}">
-      <xacro:if value="${'gazebo' in  mode}">
+      <xacro:if value="${'gazebo_classic' in  mode}">
         <gazebo>
           <plugin filename="libgazebo_ros2_control.so" name="gazebo_ros2_control">
@@ -17,4 +17,18 @@
         </gazebo>
       </xacro:if>
+      <xacro:if value="${'gazebo_classic' not in  mode}">
+        <gazebo>
+          <plugin filename="gz_ros2_control-system"
+            name="gz_ros2_control::GazeboSimROS2ControlPlugin">
+            <robot_param>robot_description</robot_param>
+            <robot_param_node>ros2_control_description</robot_param_node>
+            <parameters>${controller_manager_config_yaml_file}</parameters>
+            <!-- <hold_joints>true</hold_joints> -->
+            <ros>
+              <namespace>${ros_prefix}${base_name}</namespace>
+            </ros>
+          </plugin>
+        </gazebo>
+      </xacro:if>
     </xacro:if>
   </xacro:macro>

File: pom_description/urdf/visual/chassis.xacro (robot description, xacro)
@@ -15,8 +15,10 @@
                 <geometry>
                     <xacro:if value="${model == '4x4'}">
-                        <mesh filename="package://pom_description/meshes/pom_4x4.obj" />
+                        <!-- <mesh filename="package://pom_description/meshes/pom_4x4.obj" /> -->
+                        <mesh filename="file://$(find pom_description)/meshes/pom_4x4.obj" />
                     </xacro:if>
                     <xacro:if value="${model == 'basic'}">
-                        <mesh filename="package://pom_description/meshes/pom_basic.obj" />
+                        <!-- <mesh filename="package://pom_description/meshes/pom_basic.obj" /> -->
+                        <mesh filename="file://$(find pom_description)/meshes/pom_basic.obj" />
                     </xacro:if>
                 </geometry>

File: pom_description/urdf/visual/half_leg.xacro (robot description, xacro)
@@ -8,5 +8,6 @@
                 <origin xyz="0 0 0" rpy="0 0 0" />
                 <geometry>
-                    <mesh filename="package://pom_description/meshes/half_leg.obj" />
+                    <!-- <mesh filename="package://pom_description/meshes/half_leg.obj" /> -->
+                    <mesh filename="file://$(find pom_description)/meshes/half_leg.obj" />
                 </geometry>
                 <xacro:beige />
